Commit message: changes

File: src/kadir_description/urdf/common_properties.xacro (robot description, xacro)
@@ -7,3 +7,30 @@
         <color rgba="0.5 0.5 0.5 1" />
     </material>
+    <xacro:macro name="box_inertia" params="m l w h xyz rpy">
+        <inertial>
+            <origin xyz="${xyz}" rpy="${rpy}" />
+            <mass value="${m}" />
+            <inertia ixx="${(m/12) * (h*h + l*l)}" ixy="0" ixz="0"
+                     iyy="${(m/12) * (w*w + l*l)}" iyz="0"
+                     izz="${(m/12) * (w*w + h*h)}" />
+        </inertial>
+    </xacro:macro>
+    <xacro:macro name="cylinder_inertia" params="m r l xyz rpy">
+        <inertial>
+            <origin xyz="${xyz}" rpy="${rpy}" />
+            <mass value="${m}" />
+            <inertia ixx="${(m/12) * (3*r*r + l*l)}" ixy="0" ixz="0"
+                     iyy="${(m/12) * (3*r*r + l*l)}" iyz="0"
+                     izz="${(m/2) * (r*r)}" />
+        </inertial>
+    </xacro:macro>
+    <xacro:macro name="sphere_inertia" params="m r xyz rpy">
+        <inertial>
+            <origin xyz="${xyz}" rpy="${rpy}" />
+            <mass value="${m}" />
+            <inertia ixx="${(2*m/5) * (r*r)}" ixy="0" ixz="0"
+                     iyy="${(2*m/5) * (r*r)}" iyz="0"
+                     izz="${(2*m/5) * (r*r)}" />
+        </inertial>
+    </xacro:macro>
 </robot>

File: src/kadir_description/urdf/mobile_base.xacro (robot description, xacro)
@@ -15,4 +15,12 @@
             <material name="blue" />
         </visual>
+        <collision>
+            <geometry>
+                <box size="${base_length} ${base_width} ${base_height}" />
+            </geometry>
+            <origin xyz="0 0 ${base_height / 2.0}" rpy="0 0 0" />
+        </collision>
+        <xacro:box_inertia m = "5.0" l = "${base_length}" w = "${base_width}" h = "${base_height}"
+                            xyz = "0 0 ${base_height / 2.0}" rpy = "0 0 0" />
     </link>
     <xacro:macro name="wheel_link" params="prefix">
@@ -26,4 +34,12 @@
                 <material name="grey" />
             </visual>
+            <collision>
+                <geometry>
+                    <cylinder radius="${wheel_radius}" length="${wheel_length}" />
+                </geometry>
+                <origin xyz="0 0 0" rpy="${pi / 2.0} 0 0" />
+            </collision>
+            <xacro:cylinder_inertia m = "1.0" r = "${wheel_radius}" l = "${wheel_length}"
+                                    xyz = "0 0 0" rpy = "${pi / 2.0} 0 0" />
         </link>
     </xacro:macro>
@@ -38,4 +54,12 @@
             <material name="grey" />
         </visual>
+        <collision>
+            <geometry>
+                <sphere radius="${wheel_radius / 2.0}" />
+            </geometry>
+            <origin xyz="0 0 0" rpy="0 0 0" />
+        </collision>
+        <xacro:sphere_inertia m = "0.5" r = "${wheel_radius}"
+                                    xyz = "0 0 0" rpy = "0 0 0" />
     </link>
     <joint name="base_joint" type="fixed">
